File: hunity_tester_hat.kicad_pcb (KiCad board)
At the start: 2 copper layers, 54 x 54 mm, 16 parts, among them J1 Conn_01x10_Pin, J2 Conn_01x10_Socket, U1 experiment, U2 AP2112K-3.3

Commit message: last fixes
Parts:
- removed R1, R3: 4.7k, Resistor_SMD:R_0603_1608Metric
- JP1, JP2, JP3, JP4, JP5, JP6: moved to B.Cu
- moved JP1 38.8 mm to (101.1, 78.2)
- moved JP2 38.8 mm to (98.5, 78.2)
- moved JP3 38.8 mm to (96.0, 78.2)
- moved JP4 38.8 mm to (93.5, 78.2)
- moved JP5 38.8 mm to (90.9, 78.2)
- moved JP6 38.8 mm to (88.4, 78.2)
Routing:
- net /en: track 32.2 -> 77.1 mm, vias 2 -> 1
- net /3.3_exp: track 62.3 -> 54.0 mm
- net /sda: track 117.1 -> 110.1 mm
- net /scl: track 125.3 -> 122.5 mm
- net /en6: track 44.2 -> 43.1 mm
- net /en5: track 44.2 -> 43.1 mm
- net /en4: track 44.2 -> 43.1 mm
- net /en3: track 44.2 -> 43.1 mm
- net /en2: track 44.2 -> 43.1 mm
- net /en1: track 44.2 -> 43.1 mm
Other:
- board size 54 x 54 mm -> 56 x 54 mm
- board text removed: "1"
- board text removed: "2"
- board text removed: "3"
- board text removed: "4"
- board text removed: "5"
- board text removed: "6"
