File: hunity_tester_hat.kicad_sch (KiCad schematic)
At the start: 16 parts, among them J1 Conn_01x10_Pin, J2 Conn_01x10_Socket, U1 experiment, U2 AP2112K-3.3

Commit message: last fixes
Parts:
- removed R1, R3: 4.7k, Resistor_SMD:R_0603_1608Metric, symbol Device:R_Small
Changed lines of the file:
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@@
-	)
-	(junction
-		(at 41.91 106.68)
-		(diameter 0)
-		(color 0 0 0 0)
 	)
 	(junction
@@
 		(color 0 0 0 0)
 	)
-	(junction
-		(at 44.45 106.68)
-		(diameter 0)
-		(color 0 0 0 0)
-	)
 	(wire
 		(pts
@@
 	(wire
 		(pts
-			(xy 52.07 106.68) (xy 53.34 106.68)
-		)
-		(stroke
-			(width 0)
-			(type default)
-		)
-	)
-	(wire
-		(pts
 			(xy 111.76 41.91) (xy 111.76 43.18)
 		)
@@
 	(wire
 		(pts
-			(xy 41.91 102.87) (xy 41.91 106.68)
-		)
-		(stroke
-			(width 0)
-			(type default)
-		)
-	)
-	(wire
-		(pts
-			(xy 44.45 106.68) (xy 44.45 119.38)
+			(xy 41.91 110.49) (xy 41.91 119.38)
 		)
 		(stroke
@@
 	(wire
 		(pts
-			(xy 41.91 106.68) (xy 41.91 119.38)
-		)
-		(stroke
-			(width 0)
-			(type default)
-		)
-	)
-	(wire
-		(pts
 			(xy 36.83 114.3) (xy 36.83 119.38)
 		)
@@
 	(wire
 		(pts
-			(xy 38.1 106.68) (xy 41.91 106.68)
-		)
-		(stroke
-			(width 0)
-			(type default)
-		)
-	)
-	(wire
-		(pts
 			(xy 34.29 64.77) (xy 38.1 64.77)
 		)
@@
 	(wire
 		(pts
-			(xy 44.45 102.87) (xy 44.45 106.68)
+			(xy 44.45 110.49) (xy 44.45 119.38)
 		)
 		(stroke
@@
 	(wire
 		(pts
-			(xy 44.45 106.68) (xy 46.99 106.68)
-		)
-		(stroke
-			(width 0)
-			(type default)
-		)
-	)
-	(wire
-		(pts
 			(xy 40.64 50.8) (xy 40.64 78.74)
 		)
@@
 	(wire
 		(pts
-			(xy 31.75 106.68) (xy 33.02 106.68)
-		)
-		(stroke
-			(width 0)
-			(type default)
-		)
-	)
-	(wire
-		(pts
 			(xy 133.35 31.75) (xy 133.35 30.48)
 		)
@@
 	)
 	(label "scl"
-		(at 44.45 102.87 90)
-		(effects
-			(font
-				(size 1.27 1.27)
-			)
-			(justify left bottom)
-		)
-	)
-	(label "3.3_exp"
-		(at 53.34 106.68 0)
+		(at 44.45 110.49 90)
 		(effects
 			(font
@@
 		)
 	)
-	(label "3.3_exp"
-		(at 31.75 106.68 180)
-		(effects
-			(font
-				(size 1.27 1.27)
-			)
-			(justify right bottom)
-		)
-	)
 	(label "en4"
 		(at 29.21 114.3 90)
@@
 	)
 	(label "sda"
-		(at 41.91 102.87 90)
+		(at 41.91 110.49 90)
 		(effects
 			(font
@@
 	)
 	(symbol
-		(lib_id "Device:R_Small")
-		(at 49.53 106.68 90)
-		(unit 1)
-		(exclude_from_sim no)
-		(in_bom yes)
-		(on_board yes)
-		(dnp no)
-		(fields_autoplaced yes)
-		(property "Reference" "R3"
-			(at 49.53 101.6 90)
-			(effects
-				(font
-					(size 1.016 1.016)
-				)
-			)
-		)
-		(property "Value" "4.7k"
-			(at 49.53 104.14 90)
-			(effects
-				(font
-					(size 1.27 1.27)
-				)
-			)
-		)
-		(property "Footprint" "Resistor_SMD:R_0603_1608Metric"
-			(at 49.53 106.68 0)
-			(effects
-				(font
-					(size 1.27 1.27)
-				)
-				(hide yes)
-			)
-		)
-		(property "Datasheet" "~"
-			(at 49.53 106.68 0)
-			(effects
-				(font
-					(size 1.27 1.27)
-				)
-				(hide yes)
-			)
-		)
-		(property "Description" "Resistor, small symbol"
-			(at 49.53 106.68 0)
-			(effects
-				(font
-					(size 1.27 1.27)
-				)
-				(hide yes)
-			)
-		)
-		(pin "2"
-		)
-		(pin "1"
-		)
-		(instances
-			(project "hunity_tester_hat"
-				(path "/a2fa136e-d478-4bfa-a945-c14eb94e74a1"
-					(reference "R3")
-					(unit 1)
-				)
-			)
-		)
-	)
-	(symbol
 		(lib_id "Jumper:SolderJumper_2_Open")
 		(at 33.02 50.8 0)
@@
 					(unit 1)
 				)
-			)
-		)
-	)
-	(symbol
-		(lib_id "Device:R_Small")
-		(at 35.56 106.68 90)
-		(unit 1)
-		(exclude_from_sim no)
-		(in_bom yes)
-		(on_board yes)
-		(dnp no)
-		(fields_autoplaced yes)
-		(property "Reference" "R1"
-			(at 35.56 101.6 90)
-			(effects
-				(font
-					(size 1.016 1.016)
-				)
-			)
-		)
-		(property "Value" "4.7k"
-			(at 35.56 104.14 90)
-			(effects
-				(font
-					(size 1.27 1.27)
-				)
-			)
-		)
-		(property "Footprint" "Resistor_SMD:R_0603_1608Metric"
-			(at 35.56 106.68 0)
-			(effects
-				(font
-					(size 1.27 1.27)
-				)
-				(hide yes)
-			)
-		)
-		(property "Datasheet" "~"
-			(at 35.56 106.68 0)
-			(effects
-				(font
-					(size 1.27 1.27)
-				)
-				(hide yes)
-			)
-		)
-		(property "Description" "Resistor, small symbol"
-			(at 35.56 106.68 0)
-			(effects
-				(font
-					(size 1.27 1.27)
-				)
-				(hide yes)
-			)
-		)
-		(pin "2"
-		)
-		(pin "1"
-		)
-		(instances
-			(project ""
-				(path "/a2fa136e-d478-4bfa-a945-c14eb94e74a1"
-					(reference "R1")
-					(unit 1)
-				)
